File: kicad/mixers.kicad_sch (KiCad schematic)
At the start: 34 parts, among them U401 LM358, U402 LM358, U403 LM358

Commit message: split ch4 and ch5 connectors, update footprints
Parts:
- CD401, CD402, CD403: footprint Capacitor_SMD:C_0402_1005Metric -> Custom:C_0402_1005Metric_Fix
- RV401, RV402: footprint Connector_Wire:SolderWire-0.25sqmm_1x06_P4.2mm_D0.65mm_OD1.7mm -> Custom:ChassisMount_Wire-0.25sqmm_2x03_P4.2mm_D0.65mm_OD1.7mm
Changed lines of the file:
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@@
 			)
 		)
-		(property "Footprint" "Capacitor_SMD:C_0402_1005Metric"
+		(property "Footprint" "Custom:C_0402_1005Metric_Fix"
 			(at 213.0552 153.67 0)
 			(effects
@@
 			)
 		)
-		(property "Footprint" "Connector_Wire:SolderWire-0.25sqmm_1x06_P4.2mm_D0.65mm_OD1.7mm"
+		(property "Footprint" "Custom:ChassisMount_Wire-0.25sqmm_2x03_P4.2mm_D0.65mm_OD1.7mm"
 			(at 78.74 128.27 0)
 			(effects
@@
 			)
 		)
-		(property "Footprint" "Capacitor_SMD:C_0402_1005Metric"
+		(property "Footprint" "Custom:C_0402_1005Metric_Fix"
 			(at 187.6552 153.67 0)
 			(effects
@@
 			)
 		)
-		(property "Footprint" "Capacitor_SMD:C_0402_1005Metric"
+		(property "Footprint" "Custom:C_0402_1005Metric_Fix"
 			(at 239.7252 153.67 0)
 			(effects
@@
 			)
 		)
-		(property "Footprint" "Connector_Wire:SolderWire-0.25sqmm_1x06_P4.2mm_D0.65mm_OD1.7mm"
+		(property "Footprint" "Custom:ChassisMount_Wire-0.25sqmm_2x03_P4.2mm_D0.65mm_OD1.7mm"
 			(at 118.11 137.16 0)
 			(effects
@@
 			)
 		)
-		(property "Footprint" "Connector_Wire:SolderWire-0.25sqmm_1x06_P4.2mm_D0.65mm_OD1.7mm"
+		(property "Footprint" "Custom:ChassisMount_Wire-0.25sqmm_2x03_P4.2mm_D0.65mm_OD1.7mm"
 			(at 78.74 46.99 0)
 			(effects
@@
 			)
 		)
-		(property "Footprint" "Connector_Wire:SolderWire-0.25sqmm_1x06_P4.2mm_D0.65mm_OD1.7mm"
+		(property "Footprint" "Custom:ChassisMount_Wire-0.25sqmm_2x03_P4.2mm_D0.65mm_OD1.7mm"
 			(at 118.11 55.88 0)
 			(effects

Commit message: replace electrolytic caps with ceramics
Parts:
- removed C411, C412: 10uF, Capacitor_THT:CP_Radial_D5.0mm_P2.00mm, symbol Device:C_Polarized
- added C411, C412: 10uF, Capacitor_SMD:C_1206_3216Metric, symbol Device:C
Connections:
- net OUT.L: now also C411.1
- net OUT.R: now also C412.1
- net at U403.6 (-), U403.7: now also C412.2
- net at U403.1, U403.2 (-): now also C411.2
Changed lines of the file:
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@@
-	)
-	(symbol
-		(lib_id "Device:C_Polarized")
-		(at 144.78 52.07 180)
-		(unit 1)
-		(exclude_from_sim no)
-		(in_bom yes)
-		(on_board yes)
-		(dnp no)
-		(fields_autoplaced yes)
-		(property "Reference" "C411"
-			(at 148.59 51.6889 0)
-			(effects
-				(font
-					(size 1.27 1.27)
-				)
-				(justify right)
-			)
-		)
-		(property "Value" "10uF"
-			(at 148.59 54.2289 0)
-			(effects
-				(font
-					(size 1.27 1.27)
-				)
-				(justify right)
-			)
-		)
-		(property "Footprint" "Capacitor_THT:CP_Radial_D5.0mm_P2.00mm"
-			(at 143.8148 48.26 0)
-			(effects
-				(font
-					(size 1.27 1.27)
-				)
-				(hide yes)
-			)
-		)
-		(property "Datasheet" "~"
-			(at 144.78 52.07 0)
-			(effects
-				(font
-					(size 1.27 1.27)
-				)
-				(hide yes)
-			)
-		)
-		(property "Description" "Polarized capacitor"
-			(at 144.78 52.07 0)
-			(effects
-				(font
-					(size 1.27 1.27)
-				)
-				(hide yes)
-			)
-		)
-		(property "Supplier" "https://www.digikey.com/en/products/detail/w%C3%BCrth-elektronik/860020572003/5727172"
-			(at 144.78 52.07 0)
-			(effects
-				(font
-					(size 1.27 1.27)
-				)
-				(hide yes)
-			)
-		)
-		(pin "1"
-		)
-		(pin "2"
-		)
-		(instances
-			(project "stereo_mixer"
-				(path "/cf7176a5-9cff-4e58-aeea-84be54604336/cd4b4ef5-f327-4eb0-9bf2-427603ed98a2"
-					(reference "C411")
-					(unit 1)
-				)
-			)
-		)
 	)
 	(symbol
@@
 	)
 	(symbol
+		(lib_id "Device:C")
+		(at 144.78 133.35 0)
+		(unit 1)
+		(exclude_from_sim no)
+		(in_bom yes)
+		(on_board yes)
+		(dnp no)
+		(fields_autoplaced yes)
+		(property "Reference" "C412"
+			(at 148.59 132.0799 0)
+			(effects
+				(font
+					(size 1.27 1.27)
+				)
+				(justify left)
+			)
+		)
+		(property "Value" "10uF"
+			(at 148.59 134.6199 0)
+			(effects
+				(font
+					(size 1.27 1.27)
+				)
+				(justify left)
+			)
+		)
+		(property "Footprint" "Capacitor_SMD:C_1206_3216Metric"
+			(at 145.7452 137.16 0)
+			(effects
+				(font
+					(size 1.27 1.27)
+				)
+				(hide yes)
+			)
+		)
+		(property "Datasheet" "~"
+			(at 144.78 133.35 0)
+			(effects
+				(font
+					(size 1.27 1.27)
+				)
+				(hide yes)
+			)
+		)
+		(property "Description" "Unpolarized capacitor"
+			(at 144.78 133.35 0)
+			(effects
+				(font
+					(size 1.27 1.27)
+				)
+				(hide yes)
+			)
+		)
+		(property "Supplier" "https://www.digikey.com/en/products/detail/samsung-electro-mechanics/CL31A106KBHNNNE/3888534"
+			(at 144.78 133.35 0)
+			(effects
+				(font
+					(size 1.27 1.27)
+				)
+				(hide yes)
+			)
+		)
+		(pin "2"
+		)
+		(pin "1"
+		)
+		(instances
+			(project ""
+				(path "/cf7176a5-9cff-4e58-aeea-84be54604336/cd4b4ef5-f327-4eb0-9bf2-427603ed98a2"
+					(reference "C412")
+					(unit 1)
+				)
+			)
+		)
+	)
+	(symbol
 		(lib_id "Custom:R_Potentiometer_US_Dual_Split")
 		(at 118.11 137.16 0)
@@
 	)
 	(symbol
-		(lib_id "Device:C_Polarized")
-		(at 144.78 133.35 180)
+		(lib_id "Device:C")
+		(at 144.78 52.07 0)
 		(unit 1)
 		(exclude_from_sim no)
@@
 		(dnp no)
 		(fields_autoplaced yes)
-		(property "Reference" "C412"
-			(at 148.59 132.9689 0)
-			(effects
-				(font
-					(size 1.27 1.27)
-				)
-				(justify right)
+		(property "Reference" "C411"
+			(at 148.59 50.7999 0)
+			(effects
+				(font
+					(size 1.27 1.27)
+				)
+				(justify left)
 			)
 		)
 		(property "Value" "10uF"
-			(at 148.59 135.5089 0)
-			(effects
-				(font
-					(size 1.27 1.27)
-				)
-				(justify right)
-			)
-		)
-		(property "Footprint" "Capacitor_THT:CP_Radial_D5.0mm_P2.00mm"
-			(at 143.8148 129.54 0)
+			(at 148.59 53.3399 0)
+			(effects
+				(font
+					(size 1.27 1.27)
+				)
+				(justify left)
+			)
+		)
+		(property "Footprint" "Capacitor_SMD:C_1206_3216Metric"
+			(at 145.7452 55.88 0)
 			(effects
 				(font
@@
 		)
 		(property "Datasheet" "~"
-			(at 144.78 133.35 0)
-			(effects
-				(font
-					(size 1.27 1.27)
-				)
-				(hide yes)
-			)
-		)
-		(property "Description" "Polarized capacitor"
-			(at 144.78 133.35 0)
-			(effects
-				(font
-					(size 1.27 1.27)
-				)
-				(hide yes)
-			)
-		)
-		(property "Supplier" "https://www.digikey.com/en/products/detail/w%C3%BCrth-elektronik/860020572003/5727172"
-			(at 144.78 133.35 0)
-			(effects
-				(font
-					(size 1.27 1.27)
-				)
-				(hide yes)
-			)
-		)
-		(pin "1"
-		)
-		(pin "2"
-		)
-		(instances
-			(project "stereo_mixer"
-				(path "/cf7176a5-9cff-4e58-aeea-84be54604336/cd4b4ef5-f327-4eb0-9bf2-427603ed98a2"
-					(reference "C412")
+			(at 144.78 52.07 0)
+			(effects
+				(font
+					(size 1.27 1.27)
+				)
+				(hide yes)
+			)
+		)
+		(property "Description" "Unpolarized capacitor"
+			(at 144.78 52.07 0)
+			(effects
+				(font
+					(size 1.27 1.27)
+				)
+				(hide yes)
+			)
+		)
+		(property "Supplier" "https://www.digikey.com/en/products/detail/samsung-electro-mechanics/CL31A106KBHNNNE/3888534"
+			(at 144.78 52.07 0)
+			(effects
+				(font
+					(size 1.27 1.27)
+				)
+				(hide yes)
+			)
+		)
+		(pin "2"
+		)
+		(pin "1"
+		)
+		(instances
+			(project "stereo_mixer"
+				(path "/cf7176a5-9cff-4e58-aeea-84be54604336/cd4b4ef5-f327-4eb0-9bf2-427603ed98a2"
+					(reference "C411")
 					(unit 1)
 				)
